Commit message: Updated robot poses 'Search_ur' and 'Home_ur' and removed unused ones, updated teatcup position and stl, minor bugfix in DepthFilter

File: src/melkroboter_support/urdf/melkarm.xacro (robot description, xacro)
@@ -79,5 +79,5 @@
          <parent link="${prefix}melkarm_becherhalter" />
          <child link="${prefix}melkarm_melkbecher" />
-         <origin xyz="0.04 0.07 0" rpy="0 0 0" />
+         <origin xyz="0.04 0.07 -0.040" rpy="0 0 0" />
       </joint>
       <link name="${prefix}melkarm_melkbecher">
@@ -120,5 +120,5 @@
          <parent link="${prefix}melkarm_melkbecher" />
          <child link="${prefix}teatcup_tcp" />
-         <origin xyz="0 0 0.180" rpy="0 0 0" />
+         <origin xyz="0 0 0.170" rpy="0 0 0" />
       </joint>
       <!-- define Camera link -->
